File: kicad/TbKB.kicad_pcb (KiCad board)
At the start: 2 copper layers, 141 parts, among them U1 nice_nano

Commit message: arange pcb, switch to RP2040
Parts:
- removed Kc0r0_esc1, Kc10r0_9, Kc10r1_o1, Kc10r2_l1, Kc10r3_.1, Kc11r0_0, Kc11r1_p1, Kc11r2_;1, Kc11r3_/1, Kc11r4_Sys1, Kc13r0_del1, Kc13r4_left1, Kc14r0_-1, Kc14r1_[1, Kc14r2_'1, Kc14r3_up1, Kc14r4_down1, Kc15r0_=1, Kc15r1_]1, Kc15r2_home1, Kc15r3_end1, Kc15r4_right1, Kc1r0_tilda1, Kc1r4_fn1, Kc2r0_1, Kc2r1_q1, Kc2r2_a1, Kc2r3_z1, Kc3r0_2, Kc3r1_w1, Kc3r2_s1, Kc3r3_x1, Kc3r4_blank1, Kc4r0_3, Kc4r1_e1, Kc4r2_d1, Kc4r3_c1, Kc5r0_4, Kc5r1_r1, Kc5r2_f1, Kc5r3_v1, Kc6r0_5, Kc6r1_t1, Kc6r2_g1, Kc6r3_b1, Kc7r0_6, Kc7r1_y1, Kc7r2_h1, Kc7r3_n1, Kc8r0_7, Kc8r1_u1, Kc8r2_j1, Kc8r3_m1, Kc9r0_8, Kc9r1_i1, Kc9r2_k1, Kc9r3_,1, Kc9r4_App1, Kkc12r2_'1: SW_SPST, keyswitches:Kailh_socket_MX_1u
- removed Kc10r4_Alt1, Kc1r3_lshift1: SW_SPST, keyswitches:Kailh_socket_MX_1.25u
- removed Kc12r0_\1: SW_SPST, nice-nano-kicad:nice_nano
- removed Kc12r1_bkspc1, Kc12r3_rshift1, Kc13r2_return1: SW_SPST, keyswitches:Kailh_socket_MX_1.75u
- removed Kc1r1_tab1, Kc1r2_ctrl1, Kc2r4_super1: SW_SPST, keyswitches:Kailh_socket_MX_1.5u
- removed Kc5r4_space1: SW_SPST, keyswitches:Kailh_socket_MX
- removed Kc6r4_enter1: SW_SPST, keyswitches:Kailh_socket_MX_2.25u
- added C1: 10u, Capacitor_SMD:C_0805_2012Metric, B.Cu at (65.6, 105.2)
- added C10: 1u, Capacitor_SMD:C_0402_1005Metric, B.Cu at (61.1, 116.1)
- added C11: 100n, Capacitor_SMD:C_0402_1005Metric, B.Cu at (58.4, 109.4)
- added C12: 10u, Capacitor_SMD:C_0805_2012Metric, B.Cu at (66.2, 149.7)
- added C13: 100n, Capacitor_SMD:C_0402_1005Metric, B.Cu at (60.9, 109.4)
- added C14: 100n, Capacitor_SMD:C_0402_1005Metric, B.Cu at (53.4, 112.1)
- added C15: 100n, Capacitor_SMD:C_0402_1005Metric, B.Cu at (55.9, 112.1)
- added C16: 100n, Capacitor_SMD:C_0402_1005Metric, B.Cu at (58.4, 112.1)
- added C17: 100n, Capacitor_SMD:C_0402_1005Metric, B.Cu at (60.9, 112.1)
- added C2: 10u, Capacitor_SMD:C_0805_2012Metric, B.Cu at (67.9, 105.2)
- added C3: 100n, Capacitor_SMD:C_0402_1005Metric, B.Cu at (84.1, 125.7)
- added C4: 27p, Capacitor_SMD:C_0402_1005Metric, B.Cu at (62.1, 132.7)
- added C5: 27p, Capacitor_SMD:C_0402_1005Metric, B.Cu at (62.1, 140.5)
- added C6: 100n, Capacitor_SMD:C_0402_1005Metric, B.Cu at (53.6, 116.2)
- added C7: 100n, Capacitor_SMD:C_0402_1005Metric, B.Cu at (52.4, 116.2)
- added C8: 1u, Capacitor_SMD:C_0402_1005Metric, B.Cu at (61.1, 117.8)
- added C9: 100n, Capacitor_SMD:C_0402_1005Metric, B.Cu at (55.9, 109.4)
- added H1: MountingHole, MountingHole:MountingHole_2.2mm_M2_Pad_Via, B.Cu at (84.7, 120.7)
- added H2: MountingHole, MountingHole:MountingHole_2.2mm_M2_Pad_Via, B.Cu at (89.3, 173.2)
- added H3: MountingHole, MountingHole:MountingHole_2.2mm_M2_Pad_Via, B.Cu at (339.4, 115.9)
- added H4: MountingHole, MountingHole:MountingHole_2.2mm_M2_Pad_Via, B.Cu at (349.4, 168.4)
- added H5: MountingHole, MountingHole:MountingHole_2.2mm_M2_Pad_Via, B.Cu at (181.8, 131.6)
- added K_'1: SW_SPST, keyswitches:Kailh_socket_MX_1u, F.Cu at (329.4, 137.0)
- added K_'2: SW_SPST, keyswitches:Kailh_socket_MX_1u, F.Cu at (286.5, 137.0)
- added K_,1: SW_SPST, keyswitches:Kailh_socket_MX_1u, F.Cu at (229.4, 156.0)
- added K_-1: SW_SPST, keyswitches:Kailh_socket_MX_1u, F.Cu at (329.4, 98.9)
- added K_.1: SW_SPST, keyswitches:Kailh_socket_MX_1u, F.Cu at (248.4, 156.0)
- added K_/1: SW_SPST, keyswitches:Kailh_socket_MX_1u, F.Cu at (267.5, 156.0)
- added K_0: SW_SPST, keyswitches:Kailh_socket_MX_1u, F.Cu at (267.5, 98.9)
- added K_1: SW_SPST, keyswitches:Kailh_socket_MX_1u, F.Cu at (96.0, 98.9)
- added K_2: SW_SPST, keyswitches:Kailh_socket_MX_1u, F.Cu at (115.1, 98.9)
- added K_3: SW_SPST, keyswitches:Kailh_socket_MX_1u, F.Cu at (134.1, 98.9)
- added K_4: SW_SPST, keyswitches:Kailh_socket_MX_1u, F.Cu at (153.2, 98.9)
- added K_5: SW_SPST, keyswitches:Kailh_socket_MX_1u, F.Cu at (172.2, 98.9)
- added K_6: SW_SPST, keyswitches:Kailh_socket_MX_1u, F.Cu at (191.3, 98.9)
- added K_7: SW_SPST, keyswitches:Kailh_socket_MX_1u, F.Cu at (210.3, 98.9)
- added K_8: SW_SPST, keyswitches:Kailh_socket_MX_1u, F.Cu at (229.4, 98.9)
- added K_9: SW_SPST, keyswitches:Kailh_socket_MX_1u, F.Cu at (248.4, 98.9)
- added K_;1: SW_SPST, keyswitches:Kailh_socket_MX_1u, F.Cu at (267.5, 137.0)
- added K_=1: SW_SPST, keyswitches:Kailh_socket_MX_1u, F.Cu at (348.4, 98.9)
- added K_Alt1: SW_SPST, keyswitches:Kailh_socket_MX_1.25u, F.Cu at (246.0, 175.1)
- added K_App1: SW_SPST, keyswitches:Kailh_socket_MX_1u, F.Cu at (224.6, 175.1)
- added K_Sys1: SW_SPST, keyswitches:Kailh_socket_MX_1u, F.Cu at (267.5, 175.1)
- added K_[1: SW_SPST, keyswitches:Kailh_socket_MX_1u, F.Cu at (329.4, 117.9)
- added K_]1: SW_SPST, keyswitches:Kailh_socket_MX_1u, F.Cu at (348.4, 117.9)
- added K_a1: SW_SPST, keyswitches:Kailh_socket_MX_1u, F.Cu at (96.0, 137.0)
- added K_b1: SW_SPST, keyswitches:Kailh_socket_MX_1u, F.Cu at (172.2, 156.0)
- added K_bkslash1: SW_SPST, keyswitches:Kailh_socket_MX_1u, F.Cu at (286.5, 98.9)
- added K_bkspc1: SW_SPST, keyswitches:Kailh_socket_MX_2u, F.Cu at (296.0, 117.9)
- added K_bkspc1: SW_SPST, keyswitches:Kailh_socket_MX_1.75u, F.Cu at (293.7, 117.9)
- added K_blank1: SW_SPST, keyswitches:Kailh_socket_MX_1u, F.Cu at (124.6, 175.1)
- added K_c1: SW_SPST, keyswitches:Kailh_socket_MX_1u, F.Cu at (134.1, 156.0)
- added K_ctrl1: SW_SPST, keyswitches:Kailh_socket_MX_1.5u, F.Cu at (72.2, 137.0)
- added K_d1: SW_SPST, keyswitches:Kailh_socket_MX_1u, F.Cu at (134.1, 137.0)
- added K_del1: SW_SPST, keyswitches:Kailh_socket_MX_1u, F.Cu at (305.6, 98.9)
- added K_down1: SW_SPST, keyswitches:Kailh_socket_MX_1u, F.Cu at (324.6, 179.8)
- added K_e1: SW_SPST, keyswitches:Kailh_socket_MX_1u, F.Cu at (134.1, 117.9)
- added K_end1: SW_SPST, keyswitches:Kailh_socket_MX_1u, F.Cu at (348.4, 156.0)
- added K_enter1: SW_SPST, keyswitches:Kailh_socket_MX_2.25u, F.Cu at (193.6, 175.1)
- added K_esc1: SW_SPST, keyswitches:Kailh_socket_MX_1u, F.Cu at (57.9, 98.9)
- added K_f1: SW_SPST, keyswitches:Kailh_socket_MX_1u, F.Cu at (153.2, 137.0)
- added K_fn1: SW_SPST, keyswitches:Kailh_socket_MX_1u, F.Cu at (77.0, 175.1)
- added K_g1: SW_SPST, keyswitches:Kailh_socket_MX_1u, F.Cu at (172.2, 137.0)
- added K_h1: SW_SPST, keyswitches:Kailh_socket_MX_1u, F.Cu at (191.3, 137.0)
- added K_home1: SW_SPST, keyswitches:Kailh_socket_MX_1u, F.Cu at (348.4, 137.0)
- added K_i1: SW_SPST, keyswitches:Kailh_socket_MX_1u, F.Cu at (229.4, 117.9)
- added K_j1: SW_SPST, keyswitches:Kailh_socket_MX_1u, F.Cu at (210.3, 137.0)
- added K_k1: SW_SPST, keyswitches:Kailh_socket_MX_1u, F.Cu at (229.4, 137.0)
- added K_l1: SW_SPST, keyswitches:Kailh_socket_MX_1u, F.Cu at (248.4, 137.0)
- added K_left1: SW_SPST, keyswitches:Kailh_socket_MX_1u, F.Cu at (305.6, 179.8)
- added K_lshift1: SW_SPST, keyswitches:Kailh_socket_MX_1.25u, F.Cu at (74.6, 156.0)
- added K_m1: SW_SPST, keyswitches:Kailh_socket_MX_1u, F.Cu at (210.3, 156.0)
- added K_n1: SW_SPST, keyswitches:Kailh_socket_MX_1u, F.Cu at (191.3, 156.0)
- added K_o1: SW_SPST, keyswitches:Kailh_socket_MX_1u, F.Cu at (248.4, 117.9)
- added K_p1: SW_SPST, keyswitches:Kailh_socket_MX_1u, F.Cu at (267.5, 117.9)
- added K_q1: SW_SPST, keyswitches:Kailh_socket_MX_1u, F.Cu at (96.0, 117.9)
- added K_r1: SW_SPST, keyswitches:Kailh_socket_MX_1u, F.Cu at (153.2, 117.9)
- added K_return1: SW_SPST, keyswitches:Kailh_socket_MX_1.75u, F.Cu at (293.7, 137.0)
- added K_return1: SW_SPST, keyswitches:Kailh_socket_MX_1u, F.Cu at (305.6, 137.0)
- added K_right1: SW_SPST, keyswitches:Kailh_socket_MX_1u, F.Cu at (343.7, 179.8)
- added K_rshift1: SW_SPST, keyswitches:Kailh_socket_MX_1.75u, F.Cu at (293.7, 156.0)
- added K_rshift1: SW_SPST, keyswitches:Kailh_socket_MX_1.5u, F.Cu at (291.3, 156.0)
- added K_s1: SW_SPST, keyswitches:Kailh_socket_MX_1u, F.Cu at (115.1, 137.0)
- added K_space1: SW_SPST_3u, keyswitches:Kailh_socket_MX_1u, F.Cu at (177.0, 175.1)
- added K_space1: SW_SPST_3u, keyswitches:Kailh_socket_MX_2u, F.Cu at (153.2, 175.1)
- added K_space1: SW_SPST_3u, keyswitches:Kailh_socket_MX_1u, F.Cu at (134.1, 175.1)
- added K_super1: SW_SPST, keyswitches:Kailh_socket_MX_1.5u, F.Cu at (100.8, 175.1)
- added K_t1: SW_SPST, keyswitches:Kailh_socket_MX_1u, F.Cu at (172.2, 117.9)
- added K_tab1: SW_SPST, keyswitches:Kailh_socket_MX_1.5u, F.Cu at (72.2, 117.9)
- added K_tilda1: SW_SPST, keyswitches:Kailh_socket_MX_1u, F.Cu at (77.0, 98.9)
- added K_u1: SW_SPST, keyswitches:Kailh_socket_MX_1u, F.Cu at (210.3, 117.9)
- added K_up1: SW_SPST, keyswitches:Kailh_socket_MX_1u, F.Cu at (324.6, 160.8)
- added K_v1: SW_SPST, keyswitches:Kailh_socket_MX_1u, F.Cu at (153.2, 156.0)
- added K_w1: SW_SPST, keyswitches:Kailh_socket_MX_1u, F.Cu at (115.1, 117.9)
- added K_x1: SW_SPST, keyswitches:Kailh_socket_MX_1u, F.Cu at (115.1, 156.0)
- added K_y1: SW_SPST, keyswitches:Kailh_socket_MX_1u, F.Cu at (191.3, 117.9)
- added K_z1: SW_SPST, keyswitches:Kailh_socket_MX_1u, F.Cu at (96.0, 156.0)
- added R1: 1k, Capacitor_SMD:C_0402_1005Metric, B.Cu at (85.3, 147.5)
- added R2: 5.1k, Capacitor_SMD:C_0402_1005Metric, B.Cu at (68.4, 97.5)
- added R3: DNF, Capacitor_SMD:C_0402_1005Metric, B.Cu at (82.2, 125.6)
- added R4: 5.1k, Capacitor_SMD:C_0402_1005Metric, B.Cu at (64.9, 97.5)
- added R5: 1k, Capacitor_SMD:C_0402_1005Metric, B.Cu at (85.3, 151.2)
- added R6: 1k, Capacitor_SMD:C_0402_1005Metric, B.Cu at (62.1, 136.4)
- added R7: 27, Capacitor_SMD:C_0402_1005Metric, B.Cu at (56.3, 116.1)
- added R8: 27, Capacitor_SMD:C_0402_1005Metric, B.Cu at (58.7, 116.1)
- added SW_RST1: KMR2, Button_Switch_SMD:SW_Push_1P1T_NO_CK_KMR2, B.Cu at (81.8, 152.1)
- added SW_USB_BOOT1: KMR2, Button_Switch_SMD:SW_Push_1P1T_NO_CK_KMR2, B.Cu at (81.8, 146.6)
- added U2: W25Q128JVS, Package_SO:SOIC-8_5.23x5.23mm_P1.27mm, B.Cu at (79.3, 130.1)
- added U3: RP2040, RP2040_minimal:RP2040-QFN-56, B.Cu at (58.4, 122.9)
- added X1: USB Type C, Adafruit Feather RP2040 rev B:USB_C_CUSB31-CFM2AX-01-X, B.Cu at (66.4, 92.3)
- added Y1: ABLS-12.000MHZ-B4-T, RP2040_minimal:Crystal_SMD_HC49-US, B.Cu at (56.9, 136.7)
- D0, D1, D10, D11, D12, D13, D14, D15, D16, D17, D18, D19, D2, D20, D21, D22, D23, D24, D25, D26, D27, D28, D29, D3, D30, D31, D32, D33, D34, D35, D36, D37, D38, D39, D4, D40, D41, D42, D43, D44, D45, D46, D47, D48, D49, D5, D50, D51, D52, D53, D54, D55, D56, D57, D58, D59, D6, D60, D61, D62, D63, D64, D65, D66, D67, D68, D69, D7, D8, D9: moved to B.Cu
- U1: value nice_nano -> NCP1117-3.3_SOT223; footprint nice-nano-kicad:nice_nano -> Package_TO_SOT_SMD:SOT-223-3_TabPin2; moved to B.Cu
- moved D0 681.7 mm to (51.9, 107.9), turned to 180 degrees
- moved D9 656.4 mm to (90.0, 165.0), turned to 180 degrees
- moved D7 597.0 mm to (90.0, 126.9), turned to 180 degrees
- moved D12 589.3 mm to (109.1, 126.9), turned to 180 degrees
- moved D2 586.0 mm to (66.2, 126.9), turned to 180 degrees
- moved D1 585.9 mm to (72.4, 107.9), turned to 180 degrees
- moved D15 573.1 mm to (118.6, 184.1), turned to 180 degrees
- moved D25 568.0 mm to (166.2, 107.9), turned to 180 degrees
- moved D16 563.9 mm to (128.1, 107.9), turned to 180 degrees
- moved D18 560.3 mm to (128.1, 146.0), turned to 180 degrees
- moved D14 554.3 mm to (109.1, 165.0), turned to 180 degrees
- moved D5 551.6 mm to (71.0, 184.1), turned to 180 degrees
- moved D6 535.8 mm to (90.0, 107.9), turned to 180 degrees
- moved D27 522.6 mm to (166.2, 146.0), turned to 180 degrees
- moved D8 518.7 mm to (90.0, 146.0), turned to 180 degrees
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Connections:
- D1 pad 1: Row_0 -> Row_1
- D10 pad 1: Row_4 -> Row_8
- D11 pad 1: Row_0 -> Row_1
- D12 pad 1: Row_1 -> Row_3
- D13 pad 1: Row_2 -> Row_5
- D14 pad 1: Row_3 -> Row_7
- D15 pad 1: Row_4 -> Row_9
- D17 pad 1: Row_1 -> Row_2
- D18 pad 1: Row_2 -> Row_4
- D19 pad 1: Row_3 -> Row_6
- D2 pad 1: Row_1 -> Row_3
- D20 pad 1: Row_0 -> Row_1
- D21 pad 1: Row_1 -> Row_3
- D22 pad 1: Row_2 -> Row_5
- D23 pad 1: Row_3 -> Row_7
- D24 pad 1: Row_4 -> Row_9
- D26 pad 1: Row_1 -> Row_2
- D27 pad 1: Row_2 -> Row_4
- D28 pad 1: Row_3 -> Row_6
- D29 pad 1: Row_0 -> Row_1
- D3 pad 1: Row_2 -> Row_5
- D30 pad 1: Row_1 -> Row_3
- D31 pad 1: Row_2 -> Row_5
- D32 pad 1: Row_3 -> Row_7
- D33 pad 1: Row_4 -> Row_9
- D35 pad 1: Row_1 -> Row_2
- D36 pad 1: Row_2 -> Row_4
- D37 pad 1: Row_3 -> Row_6
- D38 pad 1: Row_0 -> Row_1
- D39 pad 1: Row_1 -> Row_3
- D4 pad 1: Row_3 -> Row_7
- D40 pad 1: Row_2 -> Row_5
- D41 pad 1: Row_3 -> Row_7
- D42 pad 1: Row_4 -> Row_9
- D44 pad 1: Row_1 -> Row_2
- D45 pad 1: Row_2 -> Row_4
- D46 pad 1: Row_3 -> Row_6
- D47 pad 1: Row_4 -> Row_8
- D48 pad 1: Row_0 -> Row_1
- D49 pad 1: Row_1 -> Row_3
- D5 pad 1: Row_4 -> Row_9
- D50 pad 1: Row_2 -> Row_5
- D51 pad 1: Row_3 -> Row_7
- D52 pad 1: Row_4 -> Row_9
- D54 pad 1: Row_1 -> Row_2
- D55 pad 1: Row_2 -> Row_4
- D56 pad 1: Row_3 -> Row_6
- D57 pad 1: Row_0 -> Row_1
- D58 pad 1: Row_2 -> Row_5
- D59 pad 1: Row_4 -> Row_9
- D61 pad 1: Row_1 -> Row_2
- D62 pad 1: Row_2 -> Row_4
- D63 pad 1: Row_3 -> Row_6
- D64 pad 1: Row_4 -> Row_8
- D65 pad 1: Row_0 -> Row_1
- D66 pad 1: Row_1 -> Row_3
- D67 pad 1: Row_2 -> Row_5
- D68 pad 1: Row_3 -> Row_7
- D69 pad 1: Row_4 -> Row_9
- D7 pad 1: Row_1 -> Row_2
- D8 pad 1: Row_2 -> Row_4
- D9 pad 1: Row_3 -> Row_6
- U1 pad 1: Col_0 -> GND
- U1 pad 2: Col_1 -> VBUS
- U1 pad 3: GND -> +3V3

Commit message: switched to smaller crystal, other switch fixes
Parts:
- K_bkspc1: footprint keyswitches:Kailh_socket_MX_1.75u -> keyswitches:Kailh_socket_MX_2u
- K_return1: footprint keyswitches:Kailh_socket_MX_1.75u -> keyswitches:Kailh_socket_MX_1u
- K_rshift1: footprint keyswitches:Kailh_socket_MX_1.75u -> keyswitches:Kailh_socket_MX_1.5u
- K_space1: footprint keyswitches:Kailh_socket_MX_2u -> keyswitches:Kailh_socket_MX_1u
- Y1: footprint RP2040_minimal:Crystal_SMD_HC49-US -> Crystal:Crystal_SMD_2520-4Pin_2.5x2.0mm
- moved R6 6.33 mm to (59.7, 130.6), turned to 90 degrees
- moved C4 5.12 mm to (57.4, 130.6), turned to 90 degrees
- moved Y1 3.45 mm to (58.4, 133.6)
Connections:
- H1 pad 1: GND -> (no net)
- H2 pad 1: GND -> (no net)
- H3 pad 1: GND -> (no net)
- H4 pad 1: GND -> (no net)
- H5 pad 1: GND -> (no net)
- U1 pad 2: VBUS -> +3V3
- U1 pad 3: +3V3 -> VBUS

Commit message: Added Addressable RGB leds, ancilarry capacitors, and edge cuts
Parts:
- added C18: 100n, Capacitor_SMD:C_0402_1005Metric, F.Cu at (129.6, 85.2)
- added C19: 100n, Capacitor_SMD:C_0402_1005Metric, B.Cu at (279.6, 104.2)
- added C20: 100n, Capacitor_SMD:C_0402_1005Metric, B.Cu at (105.8, 47.1)
- added C21: 100n, Capacitor_SMD:C_0402_1005Metric, B.Cu at (339.2, 28.0)
- added C22: 100n, Capacitor_SMD:C_0402_1005Metric, B.Cu at (91.5, 109.2)
- added C23: 100n, Capacitor_SMD:C_0402_1005Metric, B.Cu at (243.9, 28.0)
- added C24: 100n, Capacitor_SMD:C_0402_1005Metric, B.Cu at (86.7, 71.1)
- added C25: 100n, Capacitor_SMD:C_0402_1005Metric, B.Cu at (301.1, 28.0)
- added C26: 100n, Capacitor_SMD:C_0402_1005Metric, B.Cu at (167.7, 47.1)
- added C27: 100n, Capacitor_SMD:C_0402_1005Metric, B.Cu at (243.9, 85.2)
- added C28: 100n, Capacitor_SMD:C_0402_1005Metric, F.Cu at (338.5, 51.8)
- added C29: 100n, Capacitor_SMD:C_0402_1005Metric, B.Cu at (224.9, 47.1)
- added C30: 100n, Capacitor_SMD:C_0402_1005Metric, B.Cu at (105.8, 66.1)
- added C31: 100n, Capacitor_SMD:C_0402_1005Metric, B.Cu at (91.5, 28.0)
- added C32: 100n, Capacitor_SMD:C_0402_1005Metric, B.Cu at (129.6, 47.1)
- added C33: 100n, Capacitor_SMD:C_0402_1005Metric, B.Cu at (377.3, 109.0)
- added C34: 100n, Capacitor_SMD:C_0402_1005Metric, B.Cu at (363.0, 47.1)
- added C35: 100n, Capacitor_SMD:C_0402_1005Metric, B.Cu at (186.8, 85.2)
- added C36: 100n, Capacitor_SMD:C_0402_1005Metric, B.Cu at (186.8, 66.1)
- added C37: 100n, Capacitor_SMD:C_0402_1005Metric, B.Cu at (129.6, 28.0)
- added C38: 100n, Capacitor_SMD:C_0402_1005Metric, B.Cu at (224.9, 85.2)
- added C39: 100n, Capacitor_SMD:C_0402_1005Metric, B.Cu at (320.1, 28.0)
- added C40: 100n, Capacitor_SMD:C_0402_1005Metric, B.Cu at (227.2, 104.2)
- added C41: 100n, Capacitor_SMD:C_0402_1005Metric, B.Cu at (110.6, 104.2)
- added C42: 100n, Capacitor_SMD:C_0402_1005Metric, B.Cu at (301.1, 47.1)
- added C43: 100n, Capacitor_SMD:C_0402_1005Metric, B.Cu at (205.8, 28.0)
- added C44: 100n, Capacitor_SMD:C_0402_1005Metric, B.Cu at (158.2, 104.2)
- added C45: 100n, Capacitor_SMD:C_0402_1005Metric, B.Cu at (148.7, 28.0)
- added C46: 100n, Capacitor_SMD:C_0402_1005Metric, B.Cu at (282.0, 28.0)
- added C47: 100n, Capacitor_SMD:C_0402_1005Metric, B.Cu at (358.2, 109.0)
- added C48: 100n, Capacitor_SMD:C_0402_1005Metric, B.Cu at (110.6, 28.0)
- added C49: 100n, Capacitor_SMD:C_0402_1005Metric, B.Cu at (148.7, 47.1)
- added C50: 100n, Capacitor_SMD:C_0402_1005Metric, B.Cu at (205.8, 66.1)
- added C51: 100n, Capacitor_SMD:C_0402_1005Metric, B.Cu at (263.0, 66.1)
- added C52: 100n, Capacitor_SMD:C_0402_1005Metric, B.Cu at (301.1, 104.2)
- added C53: 100n, Capacitor_SMD:C_0402_1005Metric, B.Cu at (382.0, 28.0)
- added C54: 100n, Capacitor_SMD:C_0402_1005Metric, B.Cu at (282.0, 66.1)
- added C55: 100n, Capacitor_SMD:C_0402_1005Metric, B.Cu at (363.0, 66.1)
- added C56: 100n, Capacitor_SMD:C_0402_1005Metric, B.Cu at (186.8, 28.0)
- added C57: 100n, Capacitor_SMD:C_0402_1005Metric, B.Cu at (263.0, 28.0)
- added C58: 100n, Capacitor_SMD:C_0402_1005Metric, B.Cu at (363.0, 28.0)
- added C59: 100n, Capacitor_SMD:C_0402_1005Metric, B.Cu at (108.2, 85.2)
- added C60: 100n, Capacitor_SMD:C_0402_1005Metric, B.Cu at (129.6, 66.1)
- added C61: 100n, Capacitor_SMD:C_0402_1005Metric, B.Cu at (282.0, 85.2)
- added C62: 100n, Capacitor_SMD:C_0402_1005Metric, B.Cu at (358.2, 89.9)
- added C63: 100n, Capacitor_SMD:C_0402_1005Metric, B.Cu at (224.9, 28.0)
- added C64: 100n, Capacitor_SMD:C_0402_1005Metric, B.Cu at (148.7, 66.1)
- added C65: 100n, Capacitor_SMD:C_0402_1005Metric, B.Cu at (89.1, 90.2)
- added C66: 100n, Capacitor_SMD:C_0402_1005Metric, B.Cu at (243.9, 47.1)
- added C67: 100n, Capacitor_SMD:C_0402_1005Metric, B.Cu at (258.2, 104.2)
- added C68: 100n, Capacitor_SMD:C_0402_1005Metric, B.Cu at (282.0, 47.1)
- added C69: 100n, Capacitor_SMD:C_0402_1005Metric, B.Cu at (186.8, 47.1)
- added C70: 100n, Capacitor_SMD:C_0402_1005Metric, B.Cu at (205.8, 85.2)
- added C71: 100n, Capacitor_SMD:C_0402_1005Metric, B.Cu at (167.7, 66.1)
- added C72: 100n, Capacitor_SMD:C_0402_1005Metric, B.Cu at (148.7, 85.2)
- added C73: 100n, Capacitor_SMD:C_0402_1005Metric, B.Cu at (134.4, 104.2)
- added C74: 100n, Capacitor_SMD:C_0402_1005Metric, B.Cu at (330.6, 65.5)
- added C75: 100n, Capacitor_SMD:C_0402_1005Metric, B.Cu at (301.1, 85.2)
- added C76: 100n, Capacitor_SMD:C_0402_1005Metric, B.Cu at (167.7, 28.0)
- added C77: 100n, Capacitor_SMD:C_0402_1005Metric, B.Cu at (167.7, 85.2)
- added C78: 100n, Capacitor_SMD:C_0402_1005Metric, B.Cu at (301.1, 66.1)
- added C79: 100n, Capacitor_SMD:C_0402_1005Metric, B.Cu at (382.0, 66.1)
- added C80: 100n, Capacitor_SMD:C_0402_1005Metric, B.Cu at (243.9, 66.1)
- added C81: 100n, Capacitor_SMD:C_0402_1005Metric, B.Cu at (224.9, 66.1)
- added C82: 100n, Capacitor_SMD:C_0402_1005Metric, B.Cu at (382.0, 47.1)
- added C83: 100n, Capacitor_SMD:C_0402_1005Metric, B.Cu at (205.8, 47.1)
- added C84: 100n, Capacitor_SMD:C_0402_1005Metric, B.Cu at (339.2, 109.0)
- added C85: 100n, Capacitor_SMD:C_0402_1005Metric, B.Cu at (263.0, 85.2)
- added C86: 100n, Capacitor_SMD:C_0402_1005Metric, B.Cu at (263.0, 47.1)
- added C87: 100n, Capacitor_SMD:C_0402_1005Metric, B.Cu at (382.0, 85.2)
- added D100: SK6812MINI, LED_SMD:LED_SK6812MINI_PLCC4_3.5x3.5mm_P1.75mm, B.Cu at (152.4, 29.0)
- added D101: SK6812MINI, LED_SMD:LED_SK6812MINI_PLCC4_3.5x3.5mm_P1.75mm, B.Cu at (285.8, 29.0)
- added D102: SK6812MINI, LED_SMD:LED_SK6812MINI_PLCC4_3.5x3.5mm_P1.75mm, B.Cu at (133.3, 48.1)
- added D103: SK6812MINI, LED_SMD:LED_SK6812MINI_PLCC4_3.5x3.5mm_P1.75mm, B.Cu at (266.7, 48.1)
- added D104: SK6812MINI, LED_SMD:LED_SK6812MINI_PLCC4_3.5x3.5mm_P1.75mm, B.Cu at (133.3, 67.1)
- added D105: SK6812MINI, LED_SMD:LED_SK6812MINI_PLCC4_3.5x3.5mm_P1.75mm, B.Cu at (266.7, 67.1)
- added D106: SK6812MINI, LED_SMD:LED_SK6812MINI_PLCC4_3.5x3.5mm_P1.75mm, B.Cu at (133.3, 86.2)
- added D107: SK6812MINI, LED_SMD:LED_SK6812MINI_PLCC4_3.5x3.5mm_P1.75mm, B.Cu at (266.7, 86.2)
- added D108: SK6812MINI, LED_SMD:LED_SK6812MINI_PLCC4_3.5x3.5mm_P1.75mm, B.Cu at (161.9, 105.2)
- added D109: SK6812MINI, LED_SMD:LED_SK6812MINI_PLCC4_3.5x3.5mm_P1.75mm, B.Cu at (381.0, 110.0)
- added D110: SK6812MINI, LED_SMD:LED_SK6812MINI_PLCC4_3.5x3.5mm_P1.75mm, B.Cu at (171.4, 29.0)
- added D111: SK6812MINI, LED_SMD:LED_SK6812MINI_PLCC4_3.5x3.5mm_P1.75mm, B.Cu at (304.8, 29.0)
- added D112: SK6812MINI, LED_SMD:LED_SK6812MINI_PLCC4_3.5x3.5mm_P1.75mm, B.Cu at (152.4, 48.1)
- added D113: SK6812MINI, LED_SMD:LED_SK6812MINI_PLCC4_3.5x3.5mm_P1.75mm, B.Cu at (285.8, 48.1)
- added D114: SK6812MINI, LED_SMD:LED_SK6812MINI_PLCC4_3.5x3.5mm_P1.75mm, B.Cu at (152.4, 67.1)
- added D115: SK6812MINI, LED_SMD:LED_SK6812MINI_PLCC4_3.5x3.5mm_P1.75mm, B.Cu at (285.8, 67.1)
- added D116: SK6812MINI, LED_SMD:LED_SK6812MINI_PLCC4_3.5x3.5mm_P1.75mm, B.Cu at (152.4, 86.2)
- added D117: SK6812MINI, LED_SMD:LED_SK6812MINI_PLCC4_3.5x3.5mm_P1.75mm, B.Cu at (285.8, 86.2)
- added D118: SK6812MINI, LED_SMD:LED_SK6812MINI_PLCC4_3.5x3.5mm_P1.75mm, B.Cu at (231.0, 105.2)
- added D119: SK6812MINI, LED_SMD:LED_SK6812MINI_PLCC4_3.5x3.5mm_P1.75mm, B.Cu at (95.2, 110.2)
- added D120: SK6812MINI, LED_SMD:LED_SK6812MINI_PLCC4_3.5x3.5mm_P1.75mm, B.Cu at (190.5, 29.0)
- added D121: SK6812MINI, LED_SMD:LED_SK6812MINI_PLCC4_3.5x3.5mm_P1.75mm, B.Cu at (323.9, 29.0)
- added D122: SK6812MINI, LED_SMD:LED_SK6812MINI_PLCC4_3.5x3.5mm_P1.75mm, B.Cu at (171.4, 48.1)
- added D123: SK6812MINI, LED_SMD:LED_SK6812MINI_PLCC4_3.5x3.5mm_P1.75mm, B.Cu at (304.8, 48.1)
- added D124: SK6812MINI, LED_SMD:LED_SK6812MINI_PLCC4_3.5x3.5mm_P1.75mm, B.Cu at (171.4, 67.1)
- added D125: SK6812MINI, LED_SMD:LED_SK6812MINI_PLCC4_3.5x3.5mm_P1.75mm, B.Cu at (304.8, 67.1)
- added D126: SK6812MINI, LED_SMD:LED_SK6812MINI_PLCC4_3.5x3.5mm_P1.75mm, B.Cu at (171.4, 86.2)
- added D127: SK6812MINI, LED_SMD:LED_SK6812MINI_PLCC4_3.5x3.5mm_P1.75mm, B.Cu at (304.8, 86.2)
- added D128: SK6812MINI, LED_SMD:LED_SK6812MINI_PLCC4_3.5x3.5mm_P1.75mm, B.Cu at (261.9, 105.2)
- added D129: SK6812MINI, LED_SMD:LED_SK6812MINI_PLCC4_3.5x3.5mm_P1.75mm, B.Cu at (92.9, 91.2)
- added D130: SK6812MINI, LED_SMD:LED_SK6812MINI_PLCC4_3.5x3.5mm_P1.75mm, B.Cu at (209.6, 29.0)
- added D131: SK6812MINI, LED_SMD:LED_SK6812MINI_PLCC4_3.5x3.5mm_P1.75mm, B.Cu at (342.9, 29.0)
- added D132: SK6812MINI, LED_SMD:LED_SK6812MINI_PLCC4_3.5x3.5mm_P1.75mm, B.Cu at (190.5, 48.1)
- added D133: SK6812MINI, LED_SMD:LED_SK6812MINI_PLCC4_3.5x3.5mm_P1.75mm, B.Cu at (342.2, 52.8)
- added D134: SK6812MINI, LED_SMD:LED_SK6812MINI_PLCC4_3.5x3.5mm_P1.75mm, B.Cu at (190.5, 67.1)
- added D135: SK6812MINI, LED_SMD:LED_SK6812MINI_PLCC4_3.5x3.5mm_P1.75mm, B.Cu at (334.3, 66.5)
- added D136: SK6812MINI, LED_SMD:LED_SK6812MINI_PLCC4_3.5x3.5mm_P1.75mm, B.Cu at (190.5, 86.2)
- added D137: SK6812MINI, LED_SMD:LED_SK6812MINI_PLCC4_3.5x3.5mm_P1.75mm, B.Cu at (361.9, 90.9)
- added D138: SK6812MINI, LED_SMD:LED_SK6812MINI_PLCC4_3.5x3.5mm_P1.75mm, B.Cu at (283.4, 105.2)
- added D139: SK6812MINI, LED_SMD:LED_SK6812MINI_PLCC4_3.5x3.5mm_P1.75mm, B.Cu at (90.5, 72.1)
- added D70: SK6812MINI, LED_SMD:LED_SK6812MINI_PLCC4_3.5x3.5mm_P1.75mm, B.Cu at (95.2, 29.0)
- added D71: SK6812MINI, LED_SMD:LED_SK6812MINI_PLCC4_3.5x3.5mm_P1.75mm, B.Cu at (228.6, 29.0)
- added D72: SK6812MINI, LED_SMD:LED_SK6812MINI_PLCC4_3.5x3.5mm_P1.75mm, B.Cu at (366.7, 29.0)
- added D73: SK6812MINI, LED_SMD:LED_SK6812MINI_PLCC4_3.5x3.5mm_P1.75mm, B.Cu at (209.6, 48.1)
- added D74: SK6812MINI, LED_SMD:LED_SK6812MINI_PLCC4_3.5x3.5mm_P1.75mm, B.Cu at (366.7, 48.1)
- added D75: SK6812MINI, LED_SMD:LED_SK6812MINI_PLCC4_3.5x3.5mm_P1.75mm, B.Cu at (209.6, 67.1)
- added D76: SK6812MINI, LED_SMD:LED_SK6812MINI_PLCC4_3.5x3.5mm_P1.75mm, B.Cu at (366.7, 67.1)
- added D77: SK6812MINI, LED_SMD:LED_SK6812MINI_PLCC4_3.5x3.5mm_P1.75mm, B.Cu at (209.6, 86.2)
- added D78: SK6812MINI, LED_SMD:LED_SK6812MINI_PLCC4_3.5x3.5mm_P1.75mm, B.Cu at (385.8, 86.2)
- added D79: SK6812MINI, LED_SMD:LED_SK6812MINI_PLCC4_3.5x3.5mm_P1.75mm, B.Cu at (304.8, 105.2)
- added D80: SK6812MINI, LED_SMD:LED_SK6812MINI_PLCC4_3.5x3.5mm_P1.75mm, B.Cu at (114.3, 29.0)
- added D81: SK6812MINI, LED_SMD:LED_SK6812MINI_PLCC4_3.5x3.5mm_P1.75mm, B.Cu at (247.7, 29.0)
- added D82: SK6812MINI, LED_SMD:LED_SK6812MINI_PLCC4_3.5x3.5mm_P1.75mm, B.Cu at (385.8, 29.0)
- added D83: SK6812MINI, LED_SMD:LED_SK6812MINI_PLCC4_3.5x3.5mm_P1.75mm, B.Cu at (228.6, 48.1)
- added D84: SK6812MINI, LED_SMD:LED_SK6812MINI_PLCC4_3.5x3.5mm_P1.75mm, B.Cu at (385.8, 48.1)
- added D85: SK6812MINI, LED_SMD:LED_SK6812MINI_PLCC4_3.5x3.5mm_P1.75mm, B.Cu at (228.6, 67.1)
- added D86: SK6812MINI, LED_SMD:LED_SK6812MINI_PLCC4_3.5x3.5mm_P1.75mm, B.Cu at (385.8, 67.1)
- added D87: SK6812MINI, LED_SMD:LED_SK6812MINI_PLCC4_3.5x3.5mm_P1.75mm, B.Cu at (228.6, 86.2)
- added D88: SK6812MINI, LED_SMD:LED_SK6812MINI_PLCC4_3.5x3.5mm_P1.75mm, B.Cu at (114.3, 105.2)
- added D89: SK6812MINI, LED_SMD:LED_SK6812MINI_PLCC4_3.5x3.5mm_P1.75mm, B.Cu at (342.9, 110.0)
- added D90: SK6812MINI, LED_SMD:LED_SK6812MINI_PLCC4_3.5x3.5mm_P1.75mm, B.Cu at (133.3, 29.0)
- added D91: SK6812MINI, LED_SMD:LED_SK6812MINI_PLCC4_3.5x3.5mm_P1.75mm, B.Cu at (266.7, 29.0)
- added D92: SK6812MINI, LED_SMD:LED_SK6812MINI_PLCC4_3.5x3.5mm_P1.75mm, B.Cu at (109.5, 48.1)
- added D93: SK6812MINI, LED_SMD:LED_SK6812MINI_PLCC4_3.5x3.5mm_P1.75mm, B.Cu at (247.7, 48.1)
- added D94: SK6812MINI, LED_SMD:LED_SK6812MINI_PLCC4_3.5x3.5mm_P1.75mm, B.Cu at (109.5, 67.1)
- added D95: SK6812MINI, LED_SMD:LED_SK6812MINI_PLCC4_3.5x3.5mm_P1.75mm, B.Cu at (247.7, 67.1)
- added D96: SK6812MINI, LED_SMD:LED_SK6812MINI_PLCC4_3.5x3.5mm_P1.75mm, B.Cu at (111.9, 86.2)
- added D97: SK6812MINI, LED_SMD:LED_SK6812MINI_PLCC4_3.5x3.5mm_P1.75mm, B.Cu at (247.7, 86.2)
- added D98: SK6812MINI, LED_SMD:LED_SK6812MINI_PLCC4_3.5x3.5mm_P1.75mm, B.Cu at (138.1, 105.2)
- added D99: SK6812MINI, LED_SMD:LED_SK6812MINI_PLCC4_3.5x3.5mm_P1.75mm, B.Cu at (361.9, 110.0)
- added RV1: R_Potentiometer_US, potentiometers:Potentiometer_Bourns_PTA6043_Single_Slide, F.Cu at (76.2, 34.0)
- added RV2: R_Potentiometer_US, potentiometers:Potentiometer_Bourns_PTA6043_Single_Slide, F.Cu at (57.1, 34.0)
- added RV3: R_Potentiometer_US, potentiometers:Potentiometer_Bourns_PTA6043_Single_Slide, F.Cu at (38.1, 34.0)
- moved H1 86.3 mm to (123.7, 43.6)
- moved C5 81.2 mm to (97.7, 67.5)
- moved H3 81.1 mm to (376.4, 43.7)
- moved H2 80.2 mm to (123.7, 100.7)
- moved H5 78.3 mm to (219.0, 62.7)
- moved R6 77.6 mm to (103.1, 66.2)
- moved C4 77.6 mm to (100.8, 66.2)
- moved Y1 77.6 mm to (102.0, 69.3)
- moved U2 75.9 mm to (119.4, 65.7)
- moved D9 75.7 mm to (129.1, 100.2)
- moved D65 75.7 mm to (381.4, 43.0)
- moved D6 75.7 mm to (129.0, 43.0)
- moved D30 75.6 mm to (224.2, 62.1)
- moved C2 74.8 mm to (105.3, 40.4)
- moved D10 74.8 mm to (132.1, 119.2)
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Connections:
- U3 pad 37: /GPIO25 -> LED_ARRAY
- U3 pad 39: /GPIO27_ADC1 -> RV1
- U3 pad 40: /GPIO28_ADC2 -> RV2
- U3 pad 41: /GPIO29_ADC3 -> RV3
Other:
- board outline added: 368 x 104 mm

Commit message: update LEDs, USB C, stabilizers, and mounting hole placement
Parts:
- added REF**: Stabilizer_Cherry_MX_2.00u, Mounting_Keyboard_Stabilizer:Stabilizer_Cherry_MX_2.00u, F.Cu at (333.4, 53.1)
- added REF**: Stabilizer_Cherry_MX_6.25u, Mounting_Keyboard_Stabilizer:Stabilizer_Cherry_MX_6.25u, F.Cu at (214.3, 110.2)
- added REF**: Stabilizer_Cherry_MX_3.00u, Mounting_Keyboard_Stabilizer:Stabilizer_Cherry_MX_3.00u, F.Cu at (171.4, 110.2)
- added U41: CherryMX_2.25U, misc_kbd_parts:CherryMX_2.25u_PCB_Stabilizer, F.Cu at (231.0, 110.2)
- C18, C28: moved to B.Cu
- D100, D101, D102, D103, D104, D105, D106, D107, D108, D109, D110, D111, D112, D113, D114, D115, D116, D117, D118, D119, D120, D121, D122, D123, D124, D125, D126, D127, D128, D129, D130, D131, D132, D133, D134, D135, D136, D137, D138, D139, D70, D71, D72, D73, D74, D75, D76, D77, D78, D79, D80, D81, D82, D83, D84, D85, D86, D87, D88, D89, D90, D91, D92, D93, D94, D95, D96, D97, D98, D99: footprint LED_SMD:LED_SK6812MINI_PLCC4_3.5x3.5mm_P1.75mm -> keyboard_parts:LED_SK6812MINI_PLCC4_3.5x3.5mm_P1.75mm_reverse_mount; moved to F.Cu
- moved H4 77.4 mm to (294.1, 110.2)
- moved H3 32.6 mm to (345.3, 53.3)
- moved C28 21.7 mm to (316.8, 52.6), turned to 90 degrees
- moved D133 21.4 mm to (320.9, 53.9), turned to 0 degrees
- moved H2 9.87 mm to (126.2, 110.2)
- moved H1 9.72 mm to (121.4, 53.1)
- moved C3 7.75 mm to (125.0, 67.7), turned to 180 degrees
- moved D128 5.79 mm to (256.1, 105.4), turned to 0 degrees
- moved C67 5.02 mm to (253.6, 102.2)
- moved R3 3.85 mm to (123.0, 62.4), turned to 0 degrees
- moved C44 3.75 mm to (156.8, 100.8)
- moved D108 3.12 mm to (158.8, 104.7), turned to 0 degrees
- moved X1 3.05 mm to (104.5, 24.5)
- moved C20 2.37 mm to (107.5, 45.5), turned to 180 degrees
- moved D15 1.79 mm to (156.8, 120.8)
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- renumbered K_enter1 to K_Enter_2.25U, K_space1 to K_Space_2U
Other:
- outline, holes or cut-outs redrawn

Commit message: fix duplicate reference names for DSN export
Parts:
- 3U SPACE STAB: renamed from REF**
- 6.25U SPACE STAB: renamed from REF**
- renumbered REF** to 2U_STAB, K_bkspc1 to K_bkspc1_2U, K_bkspc1 to K_bkspc_1.75U, K_return1 to K_return_1.75U, K_return1 to K_return_1U, K_rshift1 to K_rshift_1.5U, K_rshift1 to K_rshift_1.75U, K_space1 to K_space_6.25U
Changed lines of the file:
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@@
     (property "Sheetname" "")
     (attr smd)
-    (fp_text reference "K_bkspc1" (at 0 -8.255) (layer "B.SilkS")
+    (fp_text reference "K_bkspc1_2U" (at 0 -8.255) (layer "B.SilkS")
       (effects (font (size 1 1) (thickness 0.15)) (justify mirror))
     )
@@
     (property "Sheetname" "")
     (attr smd)
-    (fp_text reference "K_rshift1" (at 0 -8.255 180) (layer "B.SilkS")
+    (fp_text reference "K_rshift_1.75U" (at 0 -8.255 180) (layer "B.SilkS")
       (effects (font (size 1 1) (thickness 0.15)) (justify mirror))
     )
@@
     (property "Sheetname" "")
     (attr smd)
-    (fp_text reference "K_bkspc1" (at 0 -8.255 180) (layer "B.SilkS")
+    (fp_text reference "K_bkspc_1.75U" (at 0 -8.255 180) (layer "B.SilkS")
       (effects (font (size 1 1) (thickness 0.15)) (justify mirror))
     )
@@
     (property "Sheetname" "")
     (attr smd)
-    (fp_text reference "K_space1" (at 0 -8.255) (layer "B.SilkS")
+    (fp_text reference "K_space_6.25U" (at 0 -8.255) (layer "B.SilkS")
       (effects (font (size 1 1) (thickness 0.15)) (justify mirror))
     )
@@
     (tags "Cherry MX Keyboard Stabilizer 2u 2.25u 2.5u 2.75u Cutout")
     (attr exclude_from_pos_files exclude_from_bom)
-    (fp_text reference "REF**" (at 0 -2) (layer "F.SilkS")
+    (fp_text reference "2U_STAB" (at 0 -2) (layer "F.SilkS")
       (effects (font (size 1 1) (thickness 0.15)))
     )
@@
     (property "Sheetname" "")
     (attr smd)
-    (fp_text reference "K_return1" (at 0 -8.255 180) (layer "B.SilkS")
+    (fp_text reference "K_return_1.75U" (at 0 -8.255 180) (layer "B.SilkS")
       (effects (font (size 1 1) (thickness 0.15)) (justify mirror))
     )
@@
     (property "Sheetname" "")
     (attr smd)
-    (fp_text reference "K_rshift1" (at 0 -8.255) (layer "B.SilkS")
+    (fp_text reference "K_rshift_1.5U" (at 0 -8.255) (layer "B.SilkS")
       (effects (font (size 1 1) (thickness 0.15)) (justify mirror))
     )
@@
     (tags "Cherry MX Keyboard Stabilizer 6.25u Cutout")
     (attr exclude_from_pos_files exclude_from_bom)
-    (fp_text reference "REF**" (at 0 -2) (layer "F.SilkS")
+    (fp_text reference "6.25U SPACE STAB" (at 0 -2) (layer "F.SilkS")
       (effects (font (size 1 1) (thickness 0.15)))
     )
@@
     (property "Sheetname" "")
     (attr smd)
-    (fp_text reference "K_return1" (at 0 -8.255) (layer "B.SilkS")
+    (fp_text reference "K_return_1U" (at 0 -8.255) (layer "B.SilkS")
       (effects (font (size 1 1) (thickness 0.15)) (justify mirror))
     )
@@
     (tags "Cherry MX Keyboard Stabilizer 3u Cutout")
     (attr exclude_from_pos_files exclude_from_bom)
-    (fp_text reference "REF**" (at 0 -2) (layer "F.SilkS")
+    (fp_text reference "3U SPACE STAB" (at 0 -2) (layer "F.SilkS")
       (effects (font (size 1 1) (thickness 0.15)))
     )
